Commit message: so-100 URDF 조인트 맞춤

File: tmp/so100_assets/so100.urdf (robot description, URDF)
Before this commit: robot so_arm100, 7 links, 6 joints
Links:
- link base: geometry collision mesh filename=/home/iamhjoo/myprojects/IsaacLab/tmp/so100_assets/assets/B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; visual mesh filename=/home/iamhjoo/myprojects/IsaacLab/tmp/so100_assets/assets/B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
- link gripper: geometry visual mesh filename=/home/iamhjoo/myprojects/IsaacLab/tmp/so100_assets/assets/F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; visual mesh filename=/home/iamhjoo/myprojects/IsaacLab/tmp/so100_assets/assets/F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
- link jaw: geometry visual mesh filename=/home/iamhjoo/myprojects/IsaacLab/tmp/so100_assets/assets/M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
- link lower_arm: geometry collision mesh filename=/home/iamhjoo/myprojects/IsaacLab/tmp/so100_assets/assets/L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; visual mesh filename=/home/iamhjoo/myprojects/IsaacLab/tmp/so100_assets/assets/L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
- link shoulder: geometry collision mesh filename=/home/iamhjoo/myprojects/IsaacLab/tmp/so100_assets/assets/R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; visual mesh filename=/home/iamhjoo/myprojects/IsaacLab/tmp/so100_assets/assets/R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
- link upper_arm: geometry collision mesh filename=/home/iamhjoo/myprojects/IsaacLab/tmp/so100_assets/assets/U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; visual mesh filename=/home/iamhjoo/myprojects/IsaacLab/tmp/so100_assets/assets/U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
- link wrist: geometry collision mesh filename=/home/iamhjoo/myprojects/IsaacLab/tmp/so100_assets/assets/W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; visual mesh filename=/home/iamhjoo/myprojects/IsaacLab/tmp/so100_assets/assets/W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
Joints:
- removed joint elbow_flex
- removed joint gripper
- removed joint shoulder_lift
- removed joint shoulder_pan
- removed joint wrist_flex
- removed joint wrist_roll
- added joint elbow_flex_joint: type revolute, parent upper_arm, child lower_arm, origin xyz=0 0.11257 0.028 rpy=1.57079 0 0, axis 1 0 0, limit lower=-3.14158 upper=0 effort=35 velocity=1
- added joint gripper_joint: type revolute, parent gripper, child jaw, origin xyz=-0.0202 -0.0244 0 rpy=0 3.14158 0, axis 0 0 1, limit lower=-0.2 upper=2.0 effort=35 velocity=1
- added joint shoulder_lift_joint: type revolute, parent shoulder, child upper_arm, origin xyz=0 0.1025 0.0306 rpy=-1.8 0 0, axis 1 0 0, limit lower=0 upper=3.5 effort=35 velocity=1
- added joint shoulder_pan_joint: type revolute, parent base, child shoulder, origin xyz=0 -0.0452 0.0165 rpy=1.57079 0 0, axis 0 1 0, limit lower=-2 upper=2 effort=35 velocity=1
- added joint wrist_flex_joint: type revolute, parent lower_arm, child wrist, origin xyz=0 0.0052 0.1349 rpy=-1 0 0, axis 1 0 0, limit lower=-2.5 upper=1.2 effort=35 velocity=1
- added joint wrist_roll_joint: type revolute, parent wrist, child gripper, origin xyz=0 -0.0601 0 rpy=0 1.57079 0, axis 0 1 0, limit lower=-3.14158 upper=3.14158 effort=35 velocity=1
